File: lucidGloves.kicad_pcb (KiCad board)
At the start: 2 copper layers, 73.7 x 50.8 mm, 27 parts, among them J1 USB_C_Receptacle_PowerOnly_6P, J10 Conn_01x05_Pin, J11 Conn_01x05_Pin, J12 Conn_01x19_Socket, J13 Conn_01x05_Pin, J14 Conn_01x03_Pin, J15 Conn_01x03_Pin, J16 Conn_01x03_Pin, J17 Conn_01x03_Pin, J18 Conn_01x03_Pin, J19 USB_C_Receptacle_PowerOnly_6P, J3 Conn_01x05_Pin, J4 Conn_01x05_Pin, J5 Conn_01x05_Pin, J6 Conn_01x16_Pin, J7 Conn_01x08_Pin, J8 Conn_01x19_Socket, J9 Conn_01x05_Pin, SW1 SW_Push

Commit message: Many improvements and tweaks
Parts:
- added H2: MountingHole, MountingHole:MountingHole_3.2mm_M3, F.Cu at (195.6, 91.4)
- added J14: Conn_01x06_Pin, Connector_PinHeader_2.54mm:PinHeader_1x06_P2.54mm_Horizontal, F.Cu at (180.3, 76.2)
- added J3: Conn_01x03_Pin, Connector_PinHeader_2.54mm:PinHeader_1x03_P2.54mm_Horizontal, F.Cu at (180.3, 66.0)
- D1: footprint LED_THT:LED_D5.0mm -> LED_SMD:LED_PLCC-2_3.4x3.0mm_AK
- moved G*** 26.7 mm to (161.3, 80.0)
- moved D1 13.1 mm to (168.9, 91.4), turned to 90 degrees
- moved R2 8.60 mm to (186.2, 91.4)
- moved R3 8.36 mm to (174.0, 92.7)
- moved J2 7.62 mm to (185.4, 96.5)
- moved H1 2.58 mm to (195.6, 69.8)
- moved H3 2.54 mm to (158.8, 69.8)
- moved H4 2.54 mm to (158.8, 91.4)
- moved J16 0.67 mm to (213.4, 63.5)
- moved J19 0.36 mm to (213.4, 78.7)
- moved J17 0.24 mm to (213.4, 68.6)
- moved J18 0.19 mm to (213.4, 73.7)
- moved J7 0.16 mm to (152.4, 55.9)
- renumbered H3 to H1, H5 to H3, H6 to H4, J9 to J10, J10 to J11, J11 to J12, J12 to J13, J13 to J15, J14 to J16, J15 to J17, J16 to J18, J17 to J19, J19 to J2, J18 to J20, J3 to J4, J4 to J5, J5 to J6, J6 to J7, J7 to J8, J8 to J9
Connections:
- J13 pad 13: unconnected-(J12-Pin_13-Pad13) -> Net-(J13-Pin_13)
- J13 pad 14: unconnected-(J12-Pin_14-Pad14) -> Net-(J13-Pin_14)
- J13 pad 15: unconnected-(J12-Pin_15-Pad15) -> Net-(J13-Pin_15)
- J13 pad 16: unconnected-(J12-Pin_16-Pad16) -> Net-(J13-Pin_16)
- J9 pad 12: unconnected-(J8-Pin_12-Pad12) -> Net-(J14-Pin_1)
- J9 pad 13: unconnected-(J8-Pin_13-Pad13) -> Net-(J14-Pin_2)
Routing:
- net Net-(J13-Pin_13): track 0.00 -> 34.3 mm
- net Net-(J13-Pin_16): track 0.00 -> 32.6 mm
- net Net-(J13-Pin_15): track 0.00 -> 27.1 mm
- net Net-(J13-Pin_14): track 0.00 -> 21.6 mm
- net Net-(J3-Pin_3): track 23.6 -> 39.1 mm
- net Net-(J10-Pin_5): track 150.8 -> 165.5 mm
- net Net-(J10-Pin_1): track 120.7 -> 134.9 mm
- net Net-(J14-Pin_2): track 0.00 -> 6.65 mm
- net Net-(J14-Pin_1): track 0.00 -> 6.65 mm
- net Net-(D1-K): track 10.3 -> 8.08 mm
- net Net-(J5-Pin_3): track 19.2 -> 20.9 mm
- net Net-(J2-CC1): track 4.48 -> 3.25 mm
- net Net-(D1-A): track 4.69 -> 5.33 mm
Other:
- board text added: "*"
- board text added: "*Definitely the real logo"
- board text added: "3.3V"
- board text added: "5V"
- board text added: "A"
- board text added: "B"
- board text added: "ESP32"
- board text added: "Extra pins for IO"
- board text added: "Flex1"
- board text added: "Flex2"
- board text added: "GND"
- board text added: "GPIO0"
- board text added: "GPIO12"
- board text added: "GPIO14"
- board text added: "GPIO15"
- board text added: "GPIO2"
- board text added: "GPIO4"
- board text added: "GRAB"
- board text added: "Multiplexer"
- board text added: "PWM"
- board text added: "Power"
- board text added: "SW"
- board text added: "Splay"
- board text added: "TRIG"
- board text added: "VCC"
- board text added: "X"
- board text added: "Y"
- board text added: "https://github.com/ LucidVR/lucidgloves"

Commit message: Tweaks for final JLCPCB order
Parts:
- D1: footprint LED_SMD:LED_PLCC-2_3.4x3.0mm_AK -> LED_SMD:LED_PLCC-2_3x2mm_AK
- R1, R2, R3: footprint Resistor_SMD:R_0603_1608Metric -> Resistor_SMD:R_0402_1005Metric
- moved R1 1.94 mm to (211.3, 91.4)
- moved R3 0.98 mm to (173.0, 92.7), turned to 180 degrees
Routing:
- net Net-(D1-A): track 5.33 -> 3.65 mm
- net Net-(J1-CC1): track 4.53 -> 3.05 mm
- net Net-(J16-Pin_1): track 37.1 -> 38.4 mm
